Commit message: Migrate Segway simulation from diff_drive to ros2_control effort interfaces

File: src/segway_description/urdf/segway.urdf.xacro (robot description, xacro)
@@ -16,5 +16,5 @@
   Roues : Ø65mm × 27mm
   Largeur totale : 210 + 2×27 = 264mm
-  Anti-patinage : mu1=mu2=3.0, kp=1e6, kd=100
+  Anti-patinage : mu1=mu2=1.0, kp=100000, kd=10
   ─────────────────────────────────────────────────────────────────────────────
 -->
@@ -265,4 +265,24 @@
   </joint>
   <!-- ============================================================
+       ROS 2 CONTROL — commande des roues en effort/couple
+       Les joints de roues reçoivent directement une consigne d'effort.
+       Les états position/velocity restent disponibles pour odométrie/diagnostic.
+  ============================================================ -->
+  <ros2_control name="GazeboSystem" type="system">
+    <hardware>
+      <plugin>gazebo_ros2_control/GazeboSystem</plugin>
+    </hardware>
+    <joint name="left_wheel_joint">
+      <command_interface name="effort"/>
+      <state_interface name="position"/>
+      <state_interface name="velocity"/>
+    </joint>
+    <joint name="right_wheel_joint">
+      <command_interface name="effort"/>
+      <state_interface name="position"/>
+      <state_interface name="velocity"/>
+    </joint>
+  </ros2_control>
+  <!-- ============================================================
        GAZEBO – PLUGINS ROS2 / Gazebo Classic (gazebo11)
   ============================================================ -->
@@ -276,4 +296,14 @@
     <kp>100000</kp> <kd>10</kd>
   </gazebo>
+  <!-- Plugin gazebo_ros2_control — pont Gazebo Classic ↔ ros2_control -->
+<gazebo>
+  <plugin filename="libgazebo_ros2_control.so"
+          name="gazebo_ros2_control">
+    <ros>
+      <namespace>/segway</namespace>
+    </ros>
+    <parameters>$(find segway_gazebo)/config/segway_controllers.yaml</parameters>
+  </plugin>
+</gazebo>
   <!-- Plugin joint_state_publisher -->
   <gazebo>
@@ -287,27 +317,4 @@
       <joint_name>left_wheel_joint</joint_name>
       <joint_name>right_wheel_joint</joint_name>
-    </plugin>
-  </gazebo>
-  <!-- Plugin diff_drive
-       wheel_separation = 0.210 + 0.027 = 0.237m
-       wheel_diameter   = 2 × 0.0325   = 0.065m
-  -->
-  <gazebo>
-    <plugin filename="libgazebo_ros_diff_drive.so"
-            name="diff_drive_controller">
-      <ros>
-        <namespace>/segway</namespace>
-      </ros>
-      <left_joint>left_wheel_joint</left_joint>
-      <right_joint>right_wheel_joint</right_joint>
-      <wheel_separation>0.237</wheel_separation>
-      <wheel_diameter>0.065</wheel_diameter>
-      <max_wheel_torque>2.0</max_wheel_torque>
-      <max_wheel_acceleration>10.0</max_wheel_acceleration>
-      <publish_odom>true</publish_odom>
-      <publish_odom_tf>false</publish_odom_tf>
-      <publish_wheel_tf>false</publish_wheel_tf>
-      <odometry_frame>odom</odometry_frame>
-      <robot_base_frame>base_link</robot_base_frame>
     </plugin>
   </gazebo>

Commit message: Balance controller: add vx filtering and tune outer PID
Add short moving average filter on vx.

Tune outer velocity loop with vel_kp=0.18 and vel_ki=0.01.

Improve correction of steady velocity drift.

File: src/segway_description/urdf/segway.urdf.xacro (robot description, xacro)
@@ -67,9 +67,9 @@
        MASSES (kg)
   ============================================================ -->
-  <xacro:property name="m_wheel"  value="0.040"/>  <!-- par roue -->
+  <xacro:property name="m_wheel"  value="0.120"/>  <!-- par roue -->
   <xacro:property name="m_motor"  value="0.110"/>  <!-- 2 motoréducteurs -->
   <xacro:property name="m_elec"   value="0.050"/>  <!-- pont H + convertisseurs -->
   <xacro:property name="m_cards"  value="0.050"/>  <!-- RPi + Nucleo -->
-  <xacro:property name="m_lipo"   value="0.380"/>  <!-- LiPo 3S pesée -->
+  <xacro:property name="m_lipo"   value="0.760"/>  <!-- 0.380 LiPo 3S pesée -->
   <xacro:property name="m_imu"    value="0.003"/>  <!-- MPU6050 -->
   <!-- ============================================================
@@ -318,10 +318,14 @@
   <!-- Friction roues sur sol — anti-patinage -->
   <gazebo reference="left_wheel_link">
-    <mu1>5.0</mu1>  <mu2>5.0</mu2>
-    <kp>1000000</kp> <kd>100</kd>
+<mu1>1.0</mu1>
+<mu2>1.0</mu2>
+<kp>100000</kp>
+<kd>10</kd>
   </gazebo>
   <gazebo reference="right_wheel_link">
-    <mu1>5.0</mu1>  <mu2>5.0</mu2>
-    <kp>1000000</kp> <kd>100</kd>
+<mu1>1.0</mu1>
+<mu2>1.0</mu2>
+<kp>100000</kp>
+<kd>10</kd>
   </gazebo>
   <!-- Gazebo materials -->
